Commit message: Improve husky model

File: isaac_ros/src/husky_isaac_sim/urdf/decorations.urdf.xacro (robot description, xacro)
@@ -19,4 +19,9 @@
         </geometry>
       </visual>
+      <inertial>
+          <mass value="0.01"/>
+          <origin rpy="0 0 0" xyz="0 0 0"/>
+          <inertia ixx="1.6666666666666668e-07" ixy="0" ixz="0" iyy="1.6666666666666668e-07" iyz="0" izz="1.6666666666666668e-07"/>
+      </inertial>
     </link>
     <!-- Attach chassis to the robot -->
@@ -33,4 +38,9 @@
           </geometry>
         </visual>
+      <inertial>
+          <mass value="0.01"/>
+          <origin rpy="0 0 0" xyz="0 0 0"/>
+          <inertia ixx="1.6666666666666668e-07" ixy="0" ixz="0" iyy="1.6666666666666668e-07" iyz="0" izz="1.6666666666666668e-07"/>
+      </inertial>
       </link>
       <!-- Attach user rails to base link -->
@@ -48,4 +58,9 @@
         </geometry>
       </visual>
+      <inertial>
+          <mass value="0.01"/>
+          <origin rpy="0 0 0" xyz="0 0 0"/>
+          <inertia ixx="1.6666666666666668e-07" ixy="0" ixz="0" iyy="1.6666666666666668e-07" iyz="0" izz="1.6666666666666668e-07"/>
+      </inertial>
     </link>
     <!-- Attach front bumper -->
@@ -76,4 +91,9 @@
         </geometry>
       </visual>
+      <inertial>
+          <mass value="0.01"/>
+          <origin rpy="0 0 0" xyz="0 0 0"/>
+          <inertia ixx="1.6666666666666668e-07" ixy="0" ixz="0" iyy="1.6666666666666668e-07" iyz="0" izz="1.6666666666666668e-07"/>
+      </inertial>
     </link>
     <!-- Attach rear bumper -->
@@ -113,4 +133,9 @@
             </geometry>
           </collision>
+      <inertial>
+          <mass value="0.01"/>
+          <origin rpy="0 0 0" xyz="0 0 0"/>
+          <inertia ixx="1.6666666666666668e-07" ixy="0" ixz="0" iyy="1.6666666666666668e-07" iyz="0" izz="1.6666666666666668e-07"/>
+      </inertial>
         </link>
         <!-- Attach top plate -->
@@ -167,6 +192,18 @@
         </joint>
       </xacro:unless>
-      <link name="top_plate_front_link"/>
-      <link name="top_plate_rear_link"/>
+      <link name="top_plate_front_link">
+      <inertial>
+          <mass value="0.01"/>
+          <origin rpy="0 0 0" xyz="0 0 0"/>
+          <inertia ixx="1.6666666666666668e-07" ixy="0" ixz="0" iyy="1.6666666666666668e-07" iyz="0" izz="1.6666666666666668e-07"/>
+      </inertial>
+      </link>
+      <link name="top_plate_rear_link">
+      <inertial>
+          <mass value="0.01"/>
+          <origin rpy="0 0 0" xyz="0 0 0"/>
+          <inertia ixx="1.6666666666666668e-07" ixy="0" ixz="0" iyy="1.6666666666666668e-07" iyz="0" izz="1.6666666666666668e-07"/>
+      </inertial>
+      </link>
     </xacro:if>
   </xacro:macro>

File: isaac_ros/src/husky_isaac_sim/urdf/husky.isaac.xacro (robot description, xacro)
@@ -4,37 +4,8 @@
   <!-- <xacro:arg name="name" default="" /> -->
   <xacro:arg name="prefix" default="" />
-  <xacro:arg name="gazebo_controllers" default="$(find husky_control)/config/control.yaml" />
   <xacro:arg name="path_meshes" default="package://husky_description/meshes" />
   <xacro:include filename="$(find husky_isaac_sim)/urdf/husky_macro.urdf.xacro" />
   <!-- Load husky description -->
   <xacro:husky prefix="$(arg prefix)" path_meshes="$(arg path_meshes)" />
-  <xacro:if value="$(arg is_sim)">
-    <gazebo reference="$(arg prefix)imu_link">
-      <sensor name="$(arg prefix)imu_sensor" type="imu">
-      <plugin filename="libgazebo_ros_imu_sensor.so" name="$(arg prefix)imu_plugin">
-          <ros>
-            <namespace>$(arg prefix)</namespace>
-            <remapping>~/out:=imu/data_raw</remapping>
-          </ros>
-          <initial_orientation_as_reference>false</initial_orientation_as_reference>
-        </plugin>
-        <always_on>true</always_on>
-        <update_rate>100</update_rate>
-        <visualize>true</visualize>
-      </sensor>
-    </gazebo>
-    <gazebo reference="$(arg prefix)gps_link">
-      <sensor name="$(arg prefix)gps_sensor" type="gps">
-      <plugin filename="libgazebo_ros_gps_sensor.so" name="$(arg prefix)gps_plugin">
-          <ros>
-            <namespace>$(arg prefix)</namespace>
-            <remapping>~/out:=gps/data</remapping>
-          </ros>
-        </plugin>
-        <always_on>true</always_on>
-        <update_rate>10</update_rate>
-      </sensor>
-    </gazebo>
-  </xacro:if>
   <!-- Optional custom includes. -->
   <xacro:include filename="$(arg urdf_extras)" />

File: isaac_ros/src/husky_isaac_sim/urdf/husky_macro.urdf.xacro (robot description, xacro)
@@ -13,5 +13,4 @@
   <xacro:arg name="is_sim" default="false" />
   <xacro:arg name="urdf_extras" default="$(optenv CPR_URDF_EXTRAS empty.urdf)" />
-  <xacro:arg name="serial_port" default="$(optenv HUSKY_SERIAL_PORT /dev/prolific)" />
   <!-- Included URDF/XACRO Files -->
   <xacro:include filename="$(find husky_isaac_sim)/urdf/decorations.urdf.xacro" />
@@ -45,4 +44,9 @@
         </geometry>
       </visual>
+      <inertial>
+          <mass value="0.01"/>
+          <origin rpy="0 0 0" xyz="0 0 0"/>
+          <inertia ixx="1.6666666666666668e-07" ixy="0" ixz="0" iyy="1.6666666666666668e-07" iyz="0" izz="1.6666666666666668e-07"/>
+      </inertial>
       <collision>
         <origin xyz="${( husky_front_bumper_extend - husky_rear_bumper_extend ) / 2.0} 0 ${base_z_size/4}" rpy="0 0 0" />
@@ -59,10 +63,10 @@
     </link>
     <!-- Base footprint is on the ground under the robot -->
-    <link name="${prefix}base_footprint"/>
+    <!--<link name="${prefix}base_footprint"/>
     <joint name="${prefix}base_footprint_joint" type="fixed">
       <origin xyz="0 0 ${wheel_vertical_offset - wheel_radius}" rpy="0 0 0" />
       <parent link="${prefix}base_link" />
       <child link="${prefix}base_footprint" />
-    </joint>
+    </joint>-->
     <!-- Inertial link stores the robot's inertial information -->
     <link name="${prefix}inertial_link">
@@ -80,18 +84,18 @@
     <!-- IMU Link-->
     <!-- Can be modified with environment variables in /etc/ros/setup.bash -->
-    <link name="${prefix}imu_link"/>
+    <!--<link name="${prefix}imu_link"/>
     <joint name="${prefix}imu_joint" type="fixed">
       <origin xyz="$(optenv CPR_IMU_XYZ 0 0 0)" rpy="$(optenv CPR_IMU_RPY 0 0 0)" />
       <parent link="${prefix}base_link" />
       <child link="${prefix}imu_link" />
-    </joint>
+    </joint>-->
     <!-- GPS Link-->
     <!-- Can be modified with environment variables in /etc/ros/setup.bash -->
-    <link name="${prefix}gps_link"/>
+    <!--<link name="${prefix}gps_link"/>
     <joint name="${prefix}gps_joint" type="fixed">
       <origin xyz="$(optenv CPR_GPS_XYZ 0 0 0)" rpy="$(optenv CPR_GPS_RPY 0 0 0)" />
       <parent link="${prefix}base_link" />
       <child link="${prefix}gps_link" />
-    </joint>
+    </joint>-->
     <!-- Husky wheel macros -->
     <xacro:husky_wheel wheel_prefix="${prefix}front_left">
@@ -138,54 +142,4 @@
       <xacro:intel_realsense_mount prefix="camera" topic="realsense" parent_link="realsense_mountpoint"/>
     </xacro:if>
-    <ros2_control name="${prefix}husky_hardware" type="system">
-      <hardware>
-        <xacro:if value="$(arg is_sim)">
-          <plugin>gazebo_ros2_control/GazeboSystem</plugin>
-        </xacro:if>
-        <xacro:unless value="$(arg is_sim)">
-          <plugin>husky_base/HuskyHardware</plugin>
-          <plugin>fake_components/GenericSystem</plugin>
-          <param name="hw_start_duration_sec">2.0</param>
-          <param name="hw_stop_duration_sec">3.0</param>
-          <param name="wheel_diameter">0.3302</param>
-          <param name="max_accel">5.0</param>
-          <param name="max_speed">1.0</param>
-          <param name="polling_timeout">0.1</param>
-          <param name="serial_port">$(arg serial_port)</param>
-        </xacro:unless>
-      </hardware>
-      <joint name="${prefix}front_left_wheel_joint">
-        <command_interface name="velocity">
-          <param name="min">-1</param>
-          <param name="max">1</param>
-        </command_interface>
-        <state_interface name="position"/>
-        <state_interface name="velocity"/>
-      </joint>
-      <joint name="${prefix}rear_left_wheel_joint">
-        <command_interface name="velocity">
-          <param name="min">-1</param>
-          <param name="max">1</param>
-        </command_interface>
-        <state_interface name="position"/>
-        <state_interface name="velocity"/>
-      </joint>
-      <joint name="${prefix}front_right_wheel_joint">
-        <command_interface name="velocity">
-          <param name="min">-1</param>
-          <param name="max">1</param>
-        </command_interface>
-        <state_interface name="position"/>
-        <state_interface name="velocity"/>
-      </joint>
-      <joint name="${prefix}rear_right_wheel_joint">
-        <command_interface name="velocity">
-          <param name="min">-1</param>
-          <param name="max">1</param>
-        </command_interface>
-        <state_interface name="position"/>
-        <state_interface name="velocity"/>
-      </joint>
-    </ros2_control>
   </xacro:macro>
 </robot>

File: isaac_ros/src/husky_isaac_sim/urdf/wheel.urdf.xacro (robot description, xacro)
@@ -1,5 +1,5 @@
 <?xml version="1.0"?>
 <robot xmlns:xacro="http://ros.org/wiki/xacro" name="husky_wheel">
-  <xacro:macro name="husky_wheel" params="wheel_prefix *joint_pose">
+  <xacro:macro name="husky_wheel" params="wheel_prefix *joint_pose type_rotation:=continuous">
     <link name="${wheel_prefix}_wheel">
       <inertial>
@@ -21,12 +21,5 @@
       </collision>
     </link>
-    <gazebo reference="${wheel_prefix}_wheel">
-      <mu1 value="1.0"/>
-      <mu2 value="0.5"/>
-      <kp value="10000000.0" />
-      <kd value="1.0" />
-      <fdir1 value="1 0 0"/>
-    </gazebo>
-    <joint name="${wheel_prefix}_wheel_joint" type="continuous">
+    <joint name="${wheel_prefix}_wheel_joint" type="${type_rotation}">
       <parent link="base_link"/>
       <child link="${wheel_prefix}_wheel"/>
