Commit message: Fix control Husky

File: isaac_ros/src/husky_isaac_sim/urdf/husky_macro.urdf.xacro (robot description, xacro)
@@ -44,9 +44,4 @@
         </geometry>
       </visual>
-      <inertial>
-          <mass value="0.01"/>
-          <origin rpy="0 0 0" xyz="0 0 0"/>
-          <inertia ixx="1.6666666666666668e-07" ixy="0" ixz="0" iyy="1.6666666666666668e-07" iyz="0" izz="1.6666666666666668e-07"/>
-      </inertial>
       <collision>
         <origin xyz="${( husky_front_bumper_extend - husky_rear_bumper_extend ) / 2.0} 0 ${base_z_size/4}" rpy="0 0 0" />
