Commit message: Added realsense camera

File: isaac_ros/src/husky_isaac_sim/urdf/husky.isaac.xacro (robot description, xacro)
@@ -5,7 +5,8 @@
   <xacro:arg name="prefix" default="" />
   <xacro:arg name="path_meshes" default="package://husky_description/meshes" />
+  <xacro:arg name="path_mesh_realsense" default="package://husky_isaac_sim/meshes" />
   <xacro:include filename="$(find husky_isaac_sim)/urdf/husky_macro.urdf.xacro" />
   <!-- Load husky description -->
-  <xacro:husky prefix="$(arg prefix)" path_meshes="$(arg path_meshes)" />
+  <xacro:husky prefix="$(arg prefix)" path_meshes="$(arg path_meshes)" path_mesh_realsense="$(arg path_mesh_realsense)" />
   <!-- Optional custom includes. -->
   <xacro:include filename="$(arg urdf_extras)" />

File: isaac_ros/src/husky_isaac_sim/urdf/husky_macro.urdf.xacro (robot description, xacro)
@@ -4,5 +4,5 @@
   <xacro:arg name="laser_xyz" default="$(optenv CPR_LASER_XYZ 0.2206 0.0 0.00635)" />
   <xacro:arg name="laser_rpy" default="$(optenv CPR_LASER_RPY 0.0 0.0 0.0)" />
-  <xacro:arg name="realsense_enabled" default="$(optenv CPR_REALSENSE 0)" />
+  <xacro:arg name="realsense_enabled" default="true" />
   <xacro:arg name="realsense_xyz" default="$(optenv CPR_REALSENSE_XYZ 0 0 0)" />
   <xacro:arg name="realsense_rpy" default="$(optenv CPR_REALSENSE_RPY 0 0 0)" />
@@ -16,7 +16,7 @@
   <xacro:include filename="$(find husky_isaac_sim)/urdf/decorations.urdf.xacro" />
   <xacro:include filename="$(find husky_isaac_sim)/urdf/wheel.urdf.xacro" />
-  <xacro:include filename="$(find husky_description)/urdf/accessories/intel_realsense.urdf.xacro"/>
+  <xacro:include filename="$(find husky_isaac_sim)/urdf/accessories/d435.urdf.xacro"/>
   <!-- <xacro:include filename="$(find husky_description)/urdf/accessories/sick_lms1xx_mount.urdf.xacro"/> -->
-  <xacro:include filename="$(find husky_description)/urdf/accessories/sensor_arch.urdf.xacro"/>
+  <xacro:include filename="$(find husky_isaac_sim)/urdf/accessories/sensor_arch.urdf.xacro"/>
   <xacro:property name="M_PI" value="3.14159"/>
   <!--https://github.com/ros-simulation/gazebo_ros_pkgs/pull/1284 -->
@@ -24,5 +24,5 @@
   <!--<xacro:property name="path_meshes" value="file://$(find husky_isaac_sim)/meshes"/>-->
   <!--<xacro:property name="path_meshes" value="package://husky_description/meshes"/>-->
-  <xacro:macro name="husky" params="prefix path_meshes">
+  <xacro:macro name="husky" params="prefix path_meshes path_mesh_realsense">
     <!-- Base Size -->
     <xacro:property name="base_x_size" value="0.98740000" />
@@ -121,10 +121,10 @@
       the top bar for any additional sensors in the future
     -->
-    <!-- <xacro:property name="topbar_needed_realsense" value="$(arg realsense_enabled)" />
+    <xacro:property name="topbar_needed_realsense" value="$(arg realsense_enabled)" />
     <xacro:if value="${topbar_needed_realsense}">
       <xacro:sensor_arch prefix="" parent="top_plate_link">
         <origin xyz="-0.35 0 0.51" rpy="0 0 -3.14"/>
       </xacro:sensor_arch>
-    </xacro:if> -->
+    </xacro:if>
     <!-- add the intel realsense to the topbar if needed -->
     <xacro:if value="$(arg realsense_enabled)">
@@ -135,5 +135,7 @@
         <child link="realsense_mountpoint" />
       </joint>
-      <xacro:intel_realsense_mount prefix="camera" topic="realsense" parent_link="realsense_mountpoint"/>
+      <xacro:sensor_d435 parent="realsense_mountpoint" name="camera" use_nominal_extrinsics="true" path_mesh_realsense="${path_mesh_realsense}">
+          <origin xyz="0 0 0" rpy="0 0 0" />
+      </xacro:sensor_d435>
     </xacro:if>
   </xacro:macro>

Commit message: Improve husky with ZED and fix Isaac SIM clock

File: isaac_ros/src/husky_isaac_sim/urdf/husky.isaac.xacro (robot description, xacro)
@@ -5,8 +5,8 @@
   <xacro:arg name="prefix" default="" />
   <xacro:arg name="path_meshes" default="package://husky_description/meshes" />
-  <xacro:arg name="path_mesh_realsense" default="package://husky_isaac_sim/meshes" />
+  <xacro:arg name="path_mesh_accessories" default="package://husky_isaac_sim/meshes" />
   <xacro:include filename="$(find husky_isaac_sim)/urdf/husky_macro.urdf.xacro" />
   <!-- Load husky description -->
-  <xacro:husky prefix="$(arg prefix)" path_meshes="$(arg path_meshes)" path_mesh_realsense="$(arg path_mesh_realsense)" />
+  <xacro:husky prefix="$(arg prefix)" path_meshes="$(arg path_meshes)" path_mesh_accessories="$(arg path_mesh_accessories)" />
   <!-- Optional custom includes. -->
   <xacro:include filename="$(arg urdf_extras)" />

File: isaac_ros/src/husky_isaac_sim/urdf/husky_macro.urdf.xacro (robot description, xacro)
@@ -4,8 +4,10 @@
   <xacro:arg name="laser_xyz" default="$(optenv CPR_LASER_XYZ 0.2206 0.0 0.00635)" />
   <xacro:arg name="laser_rpy" default="$(optenv CPR_LASER_RPY 0.0 0.0 0.0)" />
-  <xacro:arg name="realsense_enabled" default="true" />
+  <xacro:arg name="arch_enabled" default="true" />
+  <xacro:arg name="realsense_enabled" default="false" />
   <xacro:arg name="realsense_xyz" default="$(optenv CPR_REALSENSE_XYZ 0 0 0)" />
   <xacro:arg name="realsense_rpy" default="$(optenv CPR_REALSENSE_RPY 0 0 0)" />
   <xacro:arg name="realsense_mount" default="$(optenv CPR_REALSENSE_MOUNT_FRAME sensor_arch_mount_link)" />
+  <xacro:arg name="zed_enabled" default="true" />
   <xacro:property name="husky_front_bumper_extend" value="$(optenv HUSKY_FRONT_BUMPER_EXTEND 0)" />
   <xacro:property name="husky_rear_bumper_extend" value="$(optenv HUSKY_REAR_BUMPER_EXTEND 0)" />
@@ -17,4 +19,5 @@
   <xacro:include filename="$(find husky_isaac_sim)/urdf/wheel.urdf.xacro" />
   <xacro:include filename="$(find husky_isaac_sim)/urdf/accessories/d435.urdf.xacro"/>
+  <xacro:include filename="$(find husky_isaac_sim)/urdf/accessories/zed.urdf.xacro"/>
   <!-- <xacro:include filename="$(find husky_description)/urdf/accessories/sick_lms1xx_mount.urdf.xacro"/> -->
   <xacro:include filename="$(find husky_isaac_sim)/urdf/accessories/sensor_arch.urdf.xacro"/>
@@ -24,5 +27,5 @@
   <!--<xacro:property name="path_meshes" value="file://$(find husky_isaac_sim)/meshes"/>-->
   <!--<xacro:property name="path_meshes" value="package://husky_description/meshes"/>-->
-  <xacro:macro name="husky" params="prefix path_meshes path_mesh_realsense">
+  <xacro:macro name="husky" params="prefix path_meshes path_mesh_accessories:=package://husky_isaac_sim/meshes">
     <!-- Base Size -->
     <xacro:property name="base_x_size" value="0.98740000" />
@@ -121,5 +124,5 @@
       the top bar for any additional sensors in the future
     -->
-    <xacro:property name="topbar_needed_realsense" value="$(arg realsense_enabled)" />
+    <xacro:property name="topbar_needed_realsense" value="$(arg arch_enabled)" />
     <xacro:if value="${topbar_needed_realsense}">
       <xacro:sensor_arch prefix="" parent="top_plate_link">
@@ -139,4 +142,9 @@
       </xacro:sensor_d435>
     </xacro:if>
+    <xacro:if value="$(arg zed_enabled)">
+      <xacro:zed parent="${prefix}base_link" camera_name="zed" camera_model="zed2" path_mesh_accessories="${path_mesh_accessories}">
+          <origin xyz="-0.27 0 0.77" rpy="0 0 0" />
+      </xacro:zed>
+    </xacro:if>
   </xacro:macro>
 </robot>
