Commit message: Fix camera control and navigation

File: isaac_ros/src/husky_isaac_sim/urdf/wheel.urdf.xacro (robot description, xacro)
@@ -25,5 +25,5 @@
       <child link="${wheel_prefix}_wheel"/>
       <xacro:insert_block name="joint_pose"/>
-      <axis xyz="0 1 0" rpy="0 0 0" />
+      <axis xyz="0 -1 0" rpy="0 0 0" />
     </joint>
   </xacro:macro>

Commit message: Fix husky drive on Isaac SIM

File: isaac_ros/src/husky_isaac_sim/urdf/wheel.urdf.xacro (robot description, xacro)
@@ -25,5 +25,5 @@
       <child link="${wheel_prefix}_wheel"/>
       <xacro:insert_block name="joint_pose"/>
-      <axis xyz="0 -1 0" rpy="0 0 0" />
+      <axis xyz="0 1 0" rpy="0 0 0" />
     </joint>
   </xacro:macro>
