Commit message: Improve Husky control and camera

File: isaac_ros/src/husky_isaac_sim/urdf/accessories/zed.urdf.xacro (robot description, xacro)
@@ -106,4 +106,11 @@
             <link name="${camera_name}_temp_right_link" />
         </xacro:if>
+<!-- ZED depth -->
+        <joint name="${camera_name}_left_depth_joint" type="fixed">
+            <origin xyz="0 0 0" rpy="-${M_PI/2} 0.0 -${M_PI/2}"/>
+            <parent link="${camera_name}_left_camera_frame"/>
+            <child link="${camera_name}_left_depth_frame"/>
+        </joint>
+        <link name="${camera_name}_left_depth_frame"/>
     </xacro:macro>
 </robot>
